File: pcb/rp2040_dev.kicad_sch (KiCad schematic)
At the start: 153 parts, among them J1 USB4105-GF-A, J2 USB4105-GF-A, J3 Micro_SD_Card_Det1, J4 Conn_01x05, J5 2000-1-1-20-00-BK, J6 USB1035-GF-P-0-B-B, J7 USB1035-GF-P-0-B-B, J8 HR911105A, Q1 SI2300DS, SW1 SW_SPST_3x4mm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

Commit message: Fix UART0 reversed pins
Parts:
- BZ1: value SBZ-9032 -> Buzzer
- gave numbers to parts that had none: 4
Connections:
- net UART0_RX: now also U5.6 (TXD); no longer U5.7 (RXD)
- net UART0_TX: now also U5.7 (RXD); no longer U5.6 (TXD)
Changed lines of the file:
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@@
 (kicad_sch
-	(version 20231120)
+	(version 20250114)
 	(generator "eeschema")
-	(generator_version "8.0")
+	(generator_version "9.0")
 	(paper "User" 520 360)
+	(rectangle
+		(start 312.42 256.54)
+		(end 320.04 266.7)
+		(stroke
+			(width 0)
+			(type dash)
+		)
+		(fill
+			(type none)
+		)
+	)
+	(rectangle
+		(start 184.15 68.58)
+		(end 190.5 73.66)
+		(stroke
+			(width 0)
+			(type dash)
+		)
+		(fill
+			(type none)
+		)
+	)
+	(rectangle
+		(start 46.99 68.58)
+		(end 53.34 73.66)
+		(stroke
+			(width 0)
+			(type dash)
+		)
+		(fill
+			(type none)
+		)
+	)
+	(rectangle
+		(start 219.71 15.24)
+		(end 500.38 189.23)
+		(stroke
+			(width 1)
+			(type dash)
+		)
+		(fill
+			(type none)
+		)
+	)
+	(rectangle
+		(start 15.24 104.14)
+		(end 212.09 222.25)
+		(stroke
+			(width 1)
+			(type dash)
+		)
+		(fill
+			(type none)
+		)
+	)
+	(rectangle
+		(start 15.24 15.24)
+		(end 212.09 97.79)
+		(stroke
+			(width 1)
+			(type dash)
+		)
+		(fill
+			(type none)
+		)
+	)
+	(text "1"
+		(exclude_from_sim no)
+		(at 198.882 276.098 0)
+		(effects
+			(font
+				(size 1.27 1.27)
+				(color 255 0 0 1)
+			)
+		)
+	)
+	(text "1"
+		(exclude_from_sim no)
+		(at 198.882 280.924 0)
+		(effects
+			(font
+				(size 1.27 1.27)
+				(color 255 0 0 1)
+			)
+		)
+	)
+	(text "0"
+		(exclude_from_sim no)
+		(at 198.882 273.304 0)
+		(effects
+			(font
+				(size 1.27 1.27)
+				(color 255 0 0 1)
+			)
+		)
+	)
+	(text "1"
+		(exclude_from_sim no)
+		(at 198.882 278.384 0)
+		(effects
+			(font
+				(size 1.27 1.27)
+				(color 255 0 0 1)
+			)
+		)
+	)
+	(text "22R"
+		(exclude_from_sim no)
+		(at 316.23 254.254 0)
+		(effects
+			(font
+				(size 1.27 1.27)
+			)
+		)
+	)
+	(text "RP2040"
+		(exclude_from_sim no)
+		(at 223.52 24.13 0)
+		(effects
+			(font
+				(size 3 3)
+				(thickness 0.6)
+				(bold yes)
+			)
+			(justify left bottom)
+		)
+	)
+	(text "PHY"
+		(exclude_from_sim no)
+		(at 21.59 241.3 0)
+		(effects
+			(font
+				(size 3 3)
+				(thickness 0.6)
+				(bold yes)
+			)
+			(justify left bottom)
+		)
+	)
+	(text "USB HOST"
+		(exclude_from_sim no)
+		(at 20.32 114.3 0)
+		(effects
+			(font
+				(size 3 3)
+				(thickness 0.6)
+				(bold yes)
+			)
+			(justify left bottom)
+		)
+	)
+	(text "USB-RP"
+		(exclude_from_sim no)
+		(at 19.05 22.86 0)
+		(effects
+			(font
+				(size 3 3)
+				(thickness 0.6)
+				(bold yes)
+			)
+			(justify left bottom)
+		)
+	)
 	(junction
 		(at 101.6 266.065)
@@
 		)
 	)
-	(rectangle
-		(start 312.42 256.54)
-		(end 320.04 266.7)
-		(stroke
-			(width 0)
-			(type dash)
-		)
-		(fill
-			(type none)
-		)
-	)
-	(rectangle
-		(start 184.15 68.58)
-		(end 190.5 73.66)
-		(stroke
-			(width 0)
-			(type dash)
-		)
-		(fill
-			(type none)
-		)
-	)
-	(rectangle
-		(start 46.99 68.58)
-		(end 53.34 73.66)
-		(stroke
-			(width 0)
-			(type dash)
-		)
-		(fill
-			(type none)
-		)
-	)
-	(rectangle
-		(start 219.71 15.24)
-		(end 500.38 189.23)
-		(stroke
-			(width 1)
-			(type dash)
-		)
-		(fill
-			(type none)
-		)
-	)
-	(rectangle
-		(start 15.24 104.14)
-		(end 212.09 222.25)
-		(stroke
-			(width 1)
-			(type dash)
-		)
-		(fill
-			(type none)
-		)
-	)
-	(rectangle
-		(start 15.24 15.24)
-		(end 212.09 97.79)
-		(stroke
-			(width 1)
-			(type dash)
-		)
-		(fill
-			(type none)
-		)
-	)
-	(text "1"
-		(exclude_from_sim no)
-		(at 198.882 276.098 0)
-		(effects
-			(font
-				(size 1.27 1.27)
-				(color 255 0 0 1)
-			)
-		)
-	)
-	(text "1"
-		(exclude_from_sim no)
-		(at 198.882 280.924 0)
-		(effects
-			(font
-				(size 1.27 1.27)
-				(color 255 0 0 1)
-			)
-		)
-	)
-	(text "0"
-		(exclude_from_sim no)
-		(at 198.882 273.304 0)
-		(effects
-			(font
-				(size 1.27 1.27)
-				(color 255 0 0 1)
-			)
-		)
-	)
-	(text "1"
-		(exclude_from_sim no)
-		(at 198.882 278.384 0)
-		(effects
-			(font
-				(size 1.27 1.27)
-				(color 255 0 0 1)
-			)
-		)
-	)
-	(text "22R"
-		(exclude_from_sim no)
-		(at 316.23 254.254 0)
-		(effects
-			(font
-				(size 1.27 1.27)
-			)
-		)
-	)
-	(text "RP2040"
-		(exclude_from_sim no)
-		(at 223.52 24.13 0)
-		(effects
-			(font
-				(size 3 3)
-				(thickness 0.6)
-				(bold yes)
-			)
-			(justify left bottom)
-		)
-	)
-	(text "PHY"
-		(exclude_from_sim no)
-		(at 21.59 241.3 0)
-		(effects
-			(font
-				(size 3 3)
-				(thickness 0.6)
-				(bold yes)
-			)
-			(justify left bottom)
-		)
-	)
-	(text "USB HOST"
-		(exclude_from_sim no)
-		(at 20.32 114.3 0)
-		(effects
-			(font
-				(size 3 3)
-				(thickness 0.6)
-				(bold yes)
-			)
-			(justify left bottom)
-		)
-	)
-	(text "USB-RP"
-		(exclude_from_sim no)
-		(at 19.05 22.86 0)
-		(effects
-			(font
-				(size 3 3)
-				(thickness 0.6)
-				(bold yes)
-			)
-			(justify left bottom)
-		)
-	)
 	(label "VDDA"
 		(at 438.15 271.145 0)
@@
 	)
 	(label "UART0_TX"
-		(at 125.73 74.93 180)
+		(at 125.73 77.47 180)
 		(effects
 			(font
@@
 	)
 	(label "UART0_RX"
-		(at 125.73 77.47 180)
+		(at 125.73 74.93 180)
 		(effects
 			(font
@@
 		(dnp no)
 		(fields_autoplaced yes)
-		(property "Reference" "#PWR?"
+		(property "Reference" "#PWR018"
 			(at 30.48 82.55 0)
 			(effects
@@
 		(dnp no)
 		(fields_autoplaced yes)
-		(property "Reference" "#PWR?"
+		(property "Reference" "#PWR023"
 			(at 419.1 111.76 0)
 			(effects
@@
 		(on_board yes)
 		(dnp no)
-		(property "Reference" "R?"
+		(property "Reference" "R9"
 			(at 260.35 54.61 0)
 			(effects
@@
 		(dnp no)
 		(fields_autoplaced yes)
-		(property "Reference" "R?"
+		(property "Reference" "R2"
 			(at 381.635 23.495 90)
 			(effects
@@
 		(dnp no)
 		(fields_autoplaced yes)
-		(property "Reference" "#PWR?"
+		(property "Reference" "#PWR022"
 			(at 355.6 101.6 0)
 			(effects
@@
 		(on_board yes)
 		(dnp no)
-		(property "Reference" "R?"
+		(property "Reference" "R11"
 			(at 48.26 67.31 0)
 			(effects
@@
 			)
 		)
-		(property "Value" "SBZ-9032"
+		(property "Value" "Buzzer"
 			(at 386.08 146.6849 0)
 			(effects
@@
 		(on_board yes)
 		(dnp no)
-		(property "Reference" "R?"
+		(property "Reference" "R12"
 			(at 52.07 67.31 0)
 			(effects
@@
 		)
 	)
+	(embedded_fonts no)
 )
